File: kicad/midi-biodata-v2.kicad_pcb (KiCad board)
At the start: 2 copper layers, 90 x 45.8 mm, 43 parts, among them J1 DIN-5_180degree, J2 PJ-320B, J3 Conn_01x14_Pin, J4 PJ-320B, J5 PJ-320B, J6 PJ-320B, J7 Conn_01x02_Socket, J8 DIN-5_180degree, U1 SN74LVC1G07DBVR, U2 TLP2362TPR_E, U3 LMC555xM, U4 ESP32-S3_SUPERMINI_TH

Commit message: send v0.2 to production
Parts:
- R10: value 220 -> 220R
- R12: footprint Resistor_SMD:R_0603_1608Metric_Pad0.98x0.95mm_HandSolder -> Resistor_SMD:R_0805_2012Metric
Changed lines of the file:
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@@
 			)
 		)
-		(property "Value" "220"
+		(property "Value" "220R"
 			(at 0 1.17 0)
 			(layer "F.Fab")
@@
 		)
 	)
-	(footprint "Resistor_SMD:R_0603_1608Metric_Pad0.98x0.95mm_HandSolder"
+	(footprint "Resistor_SMD:R_0805_2012Metric"
 		(layer "F.Cu")
 		(at 43.5125 -26.2 180)
-		(descr "Resistor SMD 0603 (1608 Metric), square (rectangular) end terminal, IPC_7351 nominal with elongated pad for handsoldering. (Body size source: IPC-SM-782 page 72, https://www.pcb-3d.com/wordpress/wp-content/uploads/ipc-sm-782a_amendment_1_and_2.pdf), generated with kicad-footprint-generator")
-		(tags "resistor handsolder")
+		(descr "Resistor SMD 0805 (2012 Metric), square (rectangular) end terminal, IPC_7351 nominal, (Body size source: IPC-SM-782 page 72, https://www.pcb-3d.com/wordpress/wp-content/uploads/ipc-sm-782a_amendment_1_and_2.pdf), generated with kicad-footprint-generator")
+		(tags "resistor")
 		(property "Reference" "R12"
-			(at 0 1.6 360)
+			(at 0 -1.65 180)
 			(layer "F.SilkS")
 			(effects
@@
 		)
 		(property "Value" "470"
-			(at 0 1.43 360)
+			(at 0 1.65 180)
 			(layer "F.Fab")
 			(effects
@@
 			)
 		)
-		(property "Footprint" "Resistor_SMD:R_0603_1608Metric_Pad0.98x0.95mm_HandSolder"
+		(property "Footprint" "Resistor_SMD:R_0805_2012Metric"
 			(at 0 0 180)
 			(unlocked yes)
@@
 		(attr smd)
 		(fp_line
-			(start -0.254724 0.5225)
-			(end 0.254724 0.5225)
+			(start -0.227064 0.735)
+			(end 0.227064 0.735)
 			(stroke
 				(width 0.12)
@@
 		)
 		(fp_line
-			(start -0.254724 -0.5225)
-			(end 0.254724 -0.5225)
+			(start -0.227064 -0.735)
+			(end 0.227064 -0.735)
 			(stroke
 				(width 0.12)
@@
 		)
 		(fp_line
-			(start 1.65 0.73)
-			(end -1.65 0.73)
+			(start 1.68 0.95)
+			(end -1.68 0.95)
 			(stroke
 				(width 0.05)
@@
 		)
 		(fp_line
-			(start 1.65 -0.73)
-			(end 1.65 0.73)
+			(start 1.68 -0.95)
+			(end 1.68 0.95)
 			(stroke
 				(width 0.05)
@@
 		)
 		(fp_line
-			(start -1.65 0.73)
-			(end -1.65 -0.73)
+			(start -1.68 0.95)
+			(end -1.68 -0.95)
 			(stroke
 				(width 0.05)
@@
 		)
 		(fp_line
-			(start -1.65 -0.73)
-			(end 1.65 -0.73)
+			(start -1.68 -0.95)
+			(end 1.68 -0.95)
 			(stroke
 				(width 0.05)
@@
 		)
 		(fp_line
-			(start 0.8 0.4125)
-			(end -0.8 0.4125)
+			(start 1 0.625)
+			(end -1 0.625)
 			(stroke
 				(width 0.1)
@@
 		)
 		(fp_line
-			(start 0.8 -0.4125)
-			(end 0.8 0.4125)
+			(start 1 -0.625)
+			(end 1 0.625)
 			(stroke
 				(width 0.1)
@@
 		)
 		(fp_line
-			(start -0.8 0.4125)
-			(end -0.8 -0.4125)
+			(start -1 0.625)
+			(end -1 -0.625)
 			(stroke
 				(width 0.1)
@@
 		)
 		(fp_line
-			(start -0.8 -0.4125)
-			(end 0.8 -0.4125)
+			(start -1 -0.625)
+			(end 1 -0.625)
 			(stroke
 				(width 0.1)
@@
 		)
 		(fp_text user "${REFERENCE}"
-			(at 0 0 360)
+			(at 0 0 180)
 			(layer "F.Fab")
 			(effects
 				(font
-					(size 0.4 0.4)
-					(thickness 0.06)
+					(size 0.5 0.5)
+					(thickness 0.08)
 				)
 			)
@@
 		(pad "1" smd roundrect
 			(at -0.9125 0 180)
-			(size 0.975 0.95)
+			(size 1.025 1.4)
 			(layers "F.Cu" "F.Paste" "F.Mask")
-			(roundrect_rratio 0.25)
+			(roundrect_rratio 0.243902)
 			(net 22 "+3V3")
 			(pintype "passive")
@@
 		(pad "2" smd roundrect
 			(at 0.9125 0 180)
-			(size 0.975 0.95)
+			(size 1.025 1.4)
 			(layers "F.Cu" "F.Paste" "F.Mask")
-			(roundrect_rratio 0.25)
+			(roundrect_rratio 0.243902)
 			(net 31 "MIDI_IN")
 			(pintype "passive")
 		)
-		(model "${KICAD8_3DMODEL_DIR}/Resistor_SMD.3dshapes/R_0603_1608Metric.wrl"
+		(model "${KICAD8_3DMODEL_DIR}/Resistor_SMD.3dshapes/R_0805_2012Metric.wrl"
 			(offset
 				(xyz 0 0 0)
@@
 	)
 	(gr_text "Blue"
-		(at 49.4 -39.6 0)
+		(at 56.134 -41.148 0)
 		(layer "F.SilkS")
 		(effects
@@
 	)
 	(gr_text "GND"
-		(at 55.25 -6 0)
+		(at 61.722 -6.604 0)
 		(layer "F.SilkS")
 		(effects
@@
 	)
 	(gr_text "Vcc"
-		(at 61.5 -9 0)
+		(at 61.722 -9.144 0)
 		(layer "F.SilkS")
 		(effects
 			(font
-				(size 0.5 0.5)
-				(thickness 0.125)
+				(size 1 1)
+				(thickness 0.25)
 				(bold yes)
 			)
@@
 	)
 	(gr_text "MIDI OUT"
-		(at 5.4 -36.2 0)
+		(at 5.842 -35.56 0)
 		(layer "F.SilkS")
 		(effects
@@
 	)
 	(gr_text "GND"
-		(at 55.2 -13.8 0)
+		(at 61.722 -14.224 0)
 		(layer "F.SilkS")
 		(effects
@@
 	)
 	(gr_text "PROBE"
-		(at 51 -12.2 0)
+		(at 51.816 -12.2 0)
 		(layer "F.SilkS")
 		(effects
@@
 	)
 	(gr_text "555"
-		(at 55.2 -16.4 0)
+		(at 61.722 -16.764 0)
 		(layer "F.SilkS")
 		(effects
@@
 	)
 	(gr_text "Vcc"
-		(at 55.2 -11.2 0)
+		(at 61.722 -11.684 0)
 		(layer "F.SilkS")
 		(effects
@@
 	)
 	(gr_text "CV"
-		(at 50.4 -42.2 0)
+		(at 49.53 -41.148 0)
 		(layer "F.SilkS")
 		(effects
